Commit message: now it works

File: src/bumperbot_description/urdf/bumperbot.urdf.xacro (robot description, xacro)
@@ -7,5 +7,5 @@
             <!-- To specify the origin of the mesh -->
             <!-- The rpy (roll pitch yaw) property represents the orientation of the mesh with respect to the base link  -->
-            <!-- The xyz property describes the mesh position-->
+            <!-- The xyz property describes the mesh position respect to the base link-->
             <origin rpy="0 0 0" xyz="0 0 0"/>
             <geometry>
@@ -14,3 +14,11 @@
         </visual>
     </link>
+    <joint name="base_joint" type="fixed">
+        <!-- We will specify the parent and child link -->
+        <parent link="base_footprint"/>
+        <child link="base_link"/>
+        <!-- This states the relative position of the two links (parent and child) -->
+        <!-- We can take this info directly from the CAD model -->
+        <origin rpy="0 0 0" xyz="0 0 0.033"/>
+    </joint>
 </robot>

Commit message: updated repository

File: src/bumperbot_description/urdf/bumperbot.urdf.xacro (robot description, xacro)
@@ -22,3 +22,59 @@
         <origin rpy="0 0 0" xyz="0 0 0.033"/>
     </joint>
+    <link name="wheel_right_link">
+        <visual>
+            <origin rpy="1.57 0 0" xyz="0 0 0"/>
+            <geometry>
+                <mesh filename="package://bumperbot_description/meshes/wheel_right_link.STL"/>
+            </geometry>
+        </visual>
+    </link>
+    <joint name="wheel_right_joint" type="continuous">
+        <parent link="base_link"/>
+        <child link="wheel_right_link"/>
+        <!-- We need to say arround which axis will the wheel spin -->
+        <axis xyz="0 1 0"/>
+        <origin rpy="0 0 0" xyz="0 -0.07 0"/>
+    </joint>
+    <link name="wheel_left_link">
+        <visual>
+            <origin rpy="-1.57 0 0" xyz="0 0 0"/>
+            <geometry>
+                <mesh filename="package://bumperbot_description/meshes/wheel_left_link.STL"/>
+            </geometry>
+        </visual>
+    </link>
+    <joint name="wheel_left_joint" type="continuous">
+        <parent link="base_link"/>
+        <child link="wheel_left_link"/>
+        <!-- We need to say arround which axis will the wheel spin -->
+        <axis xyz="0 1 0"/>
+        <origin rpy="0 0 0" xyz="0 0.07 0"/>
+    </joint>
+    <link name="caster_front_link">
+        <visual>
+            <origin rpy="0 0 0" xyz="0 0 0" />
+            <geometry>
+                <mesh filename="package://bumperbot_description/meshes/caster_front_link.STL"/>
+            </geometry>
+        </visual>
+    </link>
+    <joint name="caster_front_joint" type="fixed" >
+        <parent link="base_link" />
+        <child link="caster_front_link" />
+        <origin rpy="0 0 0" xyz="0.04755 0 -0.0275" />
+    </joint>
+    <link name="caster_rear_link">
+        <visual>
+            <origin rpy="0 0 0" xyz="0 0 0" />
+            <geometry>
+                <mesh filename="package://bumperbot_description/meshes/caster_rear_link.STL"/>
+            </geometry>
+        </visual>
+    </link>
+    <joint name="caster_rear_joint" type="fixed" >
+        <parent link="base_link" />
+        <child link="caster_rear_link" />
+        <origin rpy="0 0 0" xyz="-0.04755 0 -0.0275" />
+    </joint>
 </robot>

Commit message: ?

File: src/bumperbot_description/urdf/bumperbot.urdf.xacro (robot description, xacro)
@@ -1,7 +1,15 @@
 <?xml version="1.0"?>
 <robot xmlns:xacro="http://www.ros.org/wiki/xacro" name="bumperbot">
+    <xacro:include filename="$(find bumperbot_description)/urdf/bumperbot_gazebo.xacro"/>
     <!-- This is the first link of the robot, the parent. It will be the interface between the robot and the environment -->
     <link name="base_footprint"/>
     <link name="base_link">
+        <inertial>
+            <origin xyz="0 0 0.04" rpy="0.0 0.25 0.3" />
+            <mass value="8.2573504e-01"/>
+            <inertia ixx="2.2124416e-02" ixy="-1.2294101e-04" ixz="3.4938785e-04"
+                     iyy="2.1193702e-02" iyz="-5.0120904e-05"
+                     izz="2.0064271e-02" />
+        </inertial>
         <visual>
             <!-- To specify the origin of the mesh -->
@@ -13,4 +21,10 @@
             </geometry>
         </visual>
+        <collision>
+            <origin rpy="0 0 0" xyz="0 0 0"/>
+            <geometry>
+                <mesh filename="package://bumperbot_description/meshes/base_link.STL"/>
+            </geometry>
+        </collision>
     </link>
     <joint name="base_joint" type="fixed">
@@ -23,4 +37,11 @@
     </joint>
     <link name="wheel_right_link">
+        <inertial>
+            <origin xyz="0 -0.014 0" rpy="0 0 0" />
+            <mass value="0.0530086090966721" />
+            <inertia ixx="1.88176298336665E-05" ixy="-4.8444933029987E-10" ixz="1.88163708851143E-08"
+                     iyy="3.11510738647764E-05" iyz="-6.93560663069607E-11"
+                     izz="1.8801969558182E-05" />
+        </inertial>
         <visual>
             <origin rpy="1.57 0 0" xyz="0 0 0"/>
@@ -29,4 +50,10 @@
             </geometry>
         </visual>
+        <collision>
+           <geometry>
+                <origin xyz="0 -0.015 0" rpy="1.57 0 0" />
+                <shpere radius="0.033" />
+           </geometry>
+        </collision>
     </link>
     <joint name="wheel_right_joint" type="continuous">
@@ -38,4 +65,11 @@
     </joint>
     <link name="wheel_left_link">
+        <inertial>
+            <origin xyz="0 0.014 0" rpy="0 0 0" />
+            <mass value="0.0530086043217644" />
+            <inertia ixx="1.8792911368909E-05"  ixy="3.31256392204584E-10" ixz="-1.14082001662767E-08"
+                     iyy="3.11510738759073E-05" iyz="-3.60499245082192E-10"
+                     izz="1.88266886146847E-05" />
+        </inertial>
         <visual>
             <origin rpy="-1.57 0 0" xyz="0 0 0"/>
@@ -44,4 +78,10 @@
             </geometry>
         </visual>
+        <collision>
+            <geometry>
+                 <origin xyz="0 0.015 0" rpy="1.57 0 0" />
+                 <shpere radius="0.033" />
+            </geometry>
+         </collision>
     </link>
     <joint name="wheel_left_joint" type="continuous">
@@ -53,4 +93,11 @@
     </joint>
     <link name="caster_front_link">
+        <inertial>
+            <origin xyz="3.89968128948481E-07 2.40073004698083E-07 0.00219173397061506" rpy="0 0 0" />
+            <mass value="1.44379265037903E-06" />
+            <inertia ixx="7.23075276010246E-11" ixy="-6.10956883467859E-16" ixz="2.22849693525031E-15"
+                     iyy="3.8713793085917E-11"  iyz="2.93909858781952E-15"
+                     izz="1.00967486676306E-10" />
+        </inertial>
         <visual>
             <origin rpy="0 0 0" xyz="0 0 0" />
@@ -59,4 +106,10 @@
             </geometry>
         </visual>
+        <collision>
+            <geometry>
+                 <origin xyz="0 0 0" rpy="0 0 0" />
+                 <shpere radius="0.005" />
+            </geometry>
+         </collision>
     </link>
     <joint name="caster_front_joint" type="fixed" >
@@ -66,4 +119,11 @@
     </joint>
     <link name="caster_rear_link">
+        <inertial>
+            <origin xyz="3.8996812895542E-07 2.40073004698083E-07 0.00219173397061509" rpy="0 0 0" />
+            <mass value="1.44379265037902E-06" />
+            <inertia ixx="7.23075276010246E-11" ixy="-6.10956872363424E-16" ixz="2.22849693527207E-15"
+                     iyy="3.87137930859167E-11" iyz="2.939098587861E-15"
+                     izz="1.00967486676306E-10" />
+        </inertial>
         <visual>
             <origin rpy="0 0 0" xyz="0 0 0" />
@@ -72,4 +132,10 @@
             </geometry>
         </visual>
+        <collision>
+            <geometry>
+                 <origin xyz="0 0 0" rpy="0 0 0" />
+                 <shpere radius="0.005" />
+            </geometry>
+         </collision>
     </link>
     <joint name="caster_rear_joint" type="fixed" >

Commit message: secction 4 of the nav2 course done

File: src/bumperbot_description/urdf/bumperbot.urdf.xacro (robot description, xacro)
@@ -51,8 +51,8 @@
         </visual>
         <collision>
-           <geometry>
-                <origin xyz="0 -0.015 0" rpy="1.57 0 0" />
-                <shpere radius="0.033" />
-           </geometry>
+            <origin xyz="0 -0.015 0" rpy="1.57 0 0" />
+            <geometry>
+                <sphere radius="0.033" />
+            </geometry>
         </collision>
     </link>
@@ -79,7 +79,7 @@
         </visual>
         <collision>
+            <origin xyz="0 0.015 0" rpy="1.57 0 0" />
             <geometry>
-                 <origin xyz="0 0.015 0" rpy="1.57 0 0" />
-                 <shpere radius="0.033" />
+                 <sphere radius="0.033" />
             </geometry>
          </collision>
@@ -107,7 +107,7 @@
         </visual>
         <collision>
+            <origin xyz="0 0 0" rpy="0 0 0" />
             <geometry>
-                 <origin xyz="0 0 0" rpy="0 0 0" />
-                 <shpere radius="0.005" />
+                 <sphere radius="0.005" />
             </geometry>
          </collision>
@@ -133,7 +133,7 @@
         </visual>
         <collision>
+            <origin xyz="0 0 0" rpy="0 0 0" />
             <geometry>
-                 <origin xyz="0 0 0" rpy="0 0 0" />
-                 <shpere radius="0.005" />
+                 <sphere radius="0.005" />
             </geometry>
          </collision>

Commit message: Now plugins working

File: src/bumperbot_description/urdf/bumperbot.urdf.xacro (robot description, xacro)
@@ -2,4 +2,5 @@
 <robot xmlns:xacro="http://www.ros.org/wiki/xacro" name="bumperbot">
     <xacro:include filename="$(find bumperbot_description)/urdf/bumperbot_gazebo.xacro"/>
+    <xacro:include filename="$(find bumperbot_description)/urdf/bumperbot_ros2_control.xacro"/>
     <!-- This is the first link of the robot, the parent. It will be the interface between the robot and the environment -->
     <link name="base_footprint"/>

File: src/bumperbot_description/urdf/bumperbot_gazebo.xacro (robot description, xacro)
@@ -1,4 +1,19 @@
 <?xml version="1.0"?>
 <robot name="bumperbot" xmlns:xacro="http://www.ros.org/wiki/xacro">
+    <!-- This is needed for ros2 control -->
+    <transmission name="wheel_right_transmission">
+        <plugin>transmissionInterface/SimpleTransmission</plugin>
+        <actuator name="wheel_right_motor" role="actuator_right"/>
+        <joint name="wheel_right_joint" role="joint_right">
+            <mechanical_reduction>1.0</mechanical_reduction>
+        </joint>
+    </transmission>
+    <transmission name="wheel_left_transmission">
+        <plugin>transmissionInterface/SimpleTransmission</plugin>
+        <actuator name="wheel_left_motor" role="actuator_left"/>
+        <joint name="wheel_left_joint" role="joint_left">
+            <mechanical_reduction>1.0</mechanical_reduction>
+        </joint>
+    </transmission>
     <gazebo reference="wheel_right_link">
         <mu1>100000000000000.0</mu1>
@@ -35,3 +50,10 @@
         <maxVel>0.1</maxVel>
     </gazebo>
+    <gazebo>
+        <plugin filename="libgazebo_ros2_control.so" name="gazebo_ros2_control">
+            <robot_param>robot_description</robot_param>
+            <robot_param_node>robot_state_publisher</robot_param_node>
+            <parameters>$(find bumperbot_controller)/config/bumperbot_controllers.yaml</parameters>
+        </plugin>
+    </gazebo>
 </robot>
